Commit message: fixxing cameras

File: src/mir_description/urdf/include/caster.urdf.xacro (robot description, xacro)
@@ -4,5 +4,5 @@
   <xacro:macro name="caster_wheel" params="prefix ns locationprefix locationright wheel_base_dx">
     <!-- caster hub -->
-    <joint name="${prefix}${locationprefix}_caster_rotation_joint" type="continuous">
+    <joint name="${prefix}${locationprefix}_caster_rotation_joint" type="continuous"> <!-- fixed -->
       <origin xyz="${wheel_base_dx} ${-mir_250_caster_wheel_base_dy * locationright} ${mir_250_caster_wheel_base_dz}" rpy="0 0 0" />
       <parent link="${prefix}base_link" />
@@ -51,5 +51,5 @@
     </gazebo>
     <!-- caster wheel -->
-    <joint name="${prefix}${locationprefix}_caster_wheel_joint" type="continuous">
+    <joint name="${prefix}${locationprefix}_caster_wheel_joint" type="continuous"> <!-- fixed -->
       <origin xyz="${mir_250_caster_wheel_dx} ${-mir_250_caster_wheel_dy * locationright} ${mir_250_caster_wheel_dz}" rpy="0 0 0" />
       <parent link="${prefix}${locationprefix}_caster_rotation_link" />

File: src/mir_description/urdf/include/mir_250_v1.urdf.xacro (robot description, xacro)
@@ -4,6 +4,6 @@
   <xacro:include filename="$(find mir_description)/urdf/include/imu.gazebo.urdf.xacro" />
   <xacro:include filename="$(find mir_description)/urdf/include/sick_s300.urdf.xacro" />
-  <xacro:include filename="$(find mir_description)/urdf/include/wheel.urdf.xacro" />
-  <xacro:include filename="$(find mir_description)/urdf/include/caster.urdf.xacro" />
+  <xacro:include filename="$(find mir_description)/urdf/include/wheel.urdf.xacro"/>
+  <xacro:include filename="$(find mir_description)/urdf/include/caster.urdf.xacro"/>
   <!--
   UR5e xacro files
@@ -15,4 +15,5 @@
        the bounding box and also shifted a bit to the back, because most of the mass
        is in the lower center back (because of the batteries). -->
+  <xacro:property name="wheel_separation" value="0.403"/> <!-- Distance between wheels -->
   <xacro:property name="mir_base_inertial_x" value="-0.05" />
   <xacro:property name="mir_base_inertial_y" value="0.0" />
@@ -67,4 +68,11 @@
       <material>Gazebo/Grey</material>
     </gazebo>
+    <!--
+    <link name="${prefix}odom"/>
+    <joint name="${prefix}odom_joint" type="fixed">
+      <parent link="${prefix}odom"/>
+      <child link="${prefix}base_footprint"/>
+      <origin xyz="0 0 0" rpy="0 0 0"/>
+    </joint> -->
     <!-- IMU -->
     <joint name="${prefix}base_link_to_imu_joint" type="fixed">
@@ -112,14 +120,14 @@
     <joint name="${prefix}us_1_joint" type="fixed">   <!-- right ultrasound -->
       <parent link="${prefix}base_link" />
-      <child link="${prefix}us_1_frame" />
+      <child link="${prefix}camera_floor_right_link" />
       <origin xyz="0.45 -0.12 0.16 " rpy="0 0 0" />  <!-- from visually matching to the mesh of the MiR -->
     </joint>
-    <link name="${prefix}us_1_frame" />
+    <link name="${prefix}camera_floor_right_link" />
     <joint name="${prefix}us_2_joint" type="fixed">   <!-- left ultrasound -->
       <parent link="${prefix}base_link" />
-      <child link="${prefix}us_2_frame" />
+      <child link="${prefix}camera_floor_left_link" />
       <origin xyz="0.45 0.12 0.16 " rpy="0 0 0" />  <!-- from visually matching to the mesh of the MiR -->
     </joint>
-    <link name="${prefix}us_2_frame" />
+    <link name="${prefix}camera_floor_left_link" />
     <!-- wheels -->
     <xacro:actuated_wheel prefix="${prefix}" locationprefix="left" locationright="-1"/>

File: src/mir_description/urdf/include/wheel.urdf.xacro (robot description, xacro)
@@ -2,11 +2,11 @@
 <robot xmlns:xacro="http://ros.org/wiki/xacro">
   <xacro:include filename="$(find mir_description)/urdf/include/common_properties.urdf.xacro" />
-  <xacro:macro name="actuated_wheel" params="prefix  locationprefix locationright">
-    <joint name="${prefix}${locationprefix}_wheel_joint" type="continuous">
-      <origin xyz="0.0 ${-mir_250_act_wheel_dy * locationright} ${mir_250_act_wheel_radius}" rpy="0 0 0" />
-      <parent link="${prefix}base_link" />
-      <child link="${prefix}${locationprefix}_wheel_link" />
-      <axis xyz="0 1 0" />
-      <limit effort="250" velocity="20.0" />
+  <xacro:macro name="actuated_wheel" params="prefix locationprefix locationright">
+    <joint name="${prefix}${locationprefix}_wheel_joint" type="continuous"> <!-- fixed -->
+      <origin xyz="0.0 ${-mir_250_act_wheel_dy * locationright} ${mir_250_act_wheel_radius}" rpy="0 0 0"/>
+      <parent link="${prefix}base_link"/>
+      <child link="${prefix}${locationprefix}_wheel_link"/>
+      <axis xyz="0 1 0"/>
+      <limit effort="250" velocity="20.0"/>
       <!-- <dynamics damping="0.0" friction="0.0"/> -->
       <!-- <gazebo reference="${prefix}${locationprefix}_wheel_joint">

File: src/mir_description/urdf/mir.urdf.xacro (robot description, xacro)
@@ -70,9 +70,11 @@
     </joint>
   </ros2_control>
+  <!--
   <gazebo>
-    <!-- Joint state publisher -->
     <plugin filename="libgazebo_ros2_control.so" name="gazebo_ros2_control">
       <parameters>$(find mir_description)/config/diffdrive_controller.yaml</parameters>
+      <controller_manager_node_name>controller_manager</controller_manager_node_name>
     </plugin>
   </gazebo>
+  -->
 </robot>

Commit message: Odom link works

File: src/mir_description/urdf/include/caster.urdf.xacro (robot description, xacro)
@@ -4,5 +4,5 @@
   <xacro:macro name="caster_wheel" params="prefix ns locationprefix locationright wheel_base_dx">
     <!-- caster hub -->
-    <joint name="${prefix}${locationprefix}_caster_rotation_joint" type="continuous"> <!-- fixed -->
+    <joint name="${prefix}${locationprefix}_caster_rotation_joint" type="fixed"> <!-- continuous -->
       <origin xyz="${wheel_base_dx} ${-mir_250_caster_wheel_base_dy * locationright} ${mir_250_caster_wheel_base_dz}" rpy="0 0 0" />
       <parent link="${prefix}base_link" />
@@ -51,5 +51,5 @@
     </gazebo>
     <!-- caster wheel -->
-    <joint name="${prefix}${locationprefix}_caster_wheel_joint" type="continuous"> <!-- fixed -->
+    <joint name="${prefix}${locationprefix}_caster_wheel_joint" type="fixed"> <!-- continuous -->
       <origin xyz="${mir_250_caster_wheel_dx} ${-mir_250_caster_wheel_dy * locationright} ${mir_250_caster_wheel_dz}" rpy="0 0 0" />
       <parent link="${prefix}${locationprefix}_caster_rotation_link" />

File: src/mir_description/urdf/include/wheel.urdf.xacro (robot description, xacro)
@@ -3,5 +3,5 @@
   <xacro:include filename="$(find mir_description)/urdf/include/common_properties.urdf.xacro" />
   <xacro:macro name="actuated_wheel" params="prefix locationprefix locationright">
-    <joint name="${prefix}${locationprefix}_wheel_joint" type="continuous"> <!-- fixed -->
+    <joint name="${prefix}${locationprefix}_wheel_joint" type="continuous"> <!--  fixed-->
       <origin xyz="0.0 ${-mir_250_act_wheel_dy * locationright} ${mir_250_act_wheel_radius}" rpy="0 0 0"/>
       <parent link="${prefix}base_link"/>

File: src/mir_description/urdf/mir.urdf.xacro (robot description, xacro)
@@ -14,7 +14,8 @@
   </xacro:unless>
   <xacro:mir_250 prefix="${prefix}" ns="${ns}"/>
-  <!-- <xacro:mir_ros2_control
+  <!--
+  <xacro:mir_ros2_control
     left_wheel_joint="${prefix}left_wheel_joint"
-    right_wheel_joint="${prefix}right_wheel_joint"/>  -->
+    right_wheel_joint="${prefix}right_wheel_joint"/>
   <ros2_control name="GazeboSystem" type="system">
     <hardware>
@@ -70,5 +71,4 @@
     </joint>
   </ros2_control>
-  <!--
   <gazebo>
     <plugin filename="libgazebo_ros2_control.so" name="gazebo_ros2_control">
