Commit message: CTRL+c fixxing

File: mir_description/urdf/include/mir_250_v1.urdf.xacro (robot description, xacro)
@@ -68,11 +68,4 @@
       <material>Gazebo/Grey</material>
     </gazebo>
-    <!--
-    <link name="${prefix}odom"/>
-    <joint name="${prefix}odom_joint" type="fixed">
-      <parent link="${prefix}odom"/>
-      <child link="${prefix}base_footprint"/>
-      <origin xyz="0 0 0" rpy="0 0 0"/>
-    </joint> -->
     <!-- IMU -->
     <joint name="${prefix}base_link_to_imu_joint" type="fixed">
